File: design_files/AST1014.brd (EAGLE design)
At the start: 9 x 26 mm, 15 parts, among them J1 SM05B, J2 OLED 0.69"

Commit message: updated documentation
Parts:
- removed C5: 1uF, tinycircuits:C0402
- removed R4: 1.00M, tinycircuits:0402
- removed R5: 10.0K, tinycircuits:0402
- C2: value 10uF -> 1uF
- R1: value 2K -> 10.0K
- R2: value 0.0 -> 1.00K
- R3: value 2K -> 1.00M
- moved R3 5.40 mm to (17.9, 14.8)
- moved R1 3.98 mm to (14.7, 18.5), turned to 180 degrees
- moved C1 2.24 mm to (14.8, 20.7)
- moved C2 2.24 mm to (11.8, 17.6)
- moved C3 2.24 mm to (10.7, 19.9)
- moved C4 2.24 mm to (13.0, 19.9)
- moved C6 2.24 mm to (16.8, 19.8)
- moved C7 2.24 mm to (18.3, 20.2)
- moved J1 2.24 mm to (14.5, 10.3)
- moved J2 2.24 mm to (14.5, 27.6)
- moved R2 2.24 mm to (16.5, 15.7)
Connections:
- net GND: now also R3.1; no longer C5.2, R4.1
- net N$10: now also R1.1; no longer R5.1
- net N$8: now also R3.2; no longer R4.2
- net SCL: no longer R3.1
- net SDA: no longer R1.1
- net VCC: no longer C5.1, R3.2, R5.2
Routing:
- net VCC: track 23.5 -> 20.0 mm
- net SCL: track 18.3 -> 17.5 mm
- net SDA: track 17.4 -> 16.6 mm
Other:
- board text added: "AST1014 R1"
- board text added: "Wireling 0.69 OLED"
- board text removed: "Screen R1"
