File: design_files/AST1014.sch (EAGLE design)
At the start: 14 parts, among them J1 SM05B, J2 OLED 0.69"

Commit message: updated documentation
Parts:
- removed C5: 1uF, tinycircuits:AS-ITM-00105
- removed R4: 1.00M, tinycircuits:AS-ITM-00005
- removed R5: 10.0K, tinycircuits:AS-ITM-00032
- C2: value 10uF -> 1uF; device tinycircuits:AS-ITM-00002 -> tinycircuits:AS-ITM-00347; PARTNO (none) -> AS-ITM-00347; VALUE (none) -> 1uF
- R1: value 2K -> 10.0K; device tinycircuits:AS-ITM-00315 -> tinycircuits:AS-ITM-00032
- R2: value 0.0 -> 1.00K; device tinycircuits:AS-ITM-00076 -> tinycircuits:AS-ITM-00003; PARTNO (none) -> AS-ITM-00003; VALUE (none) -> 1.00K
- R3: value 2K -> 1.00M; device tinycircuits:AS-ITM-00315 -> tinycircuits:AS-ITM-00005
Connections:
- net GND: now also R3.1; no longer C5.2, R4.1
- net N$10: now also R1.1; no longer R5.1
- net N$8: now also R3.2; no longer R4.2
- net SCL: no longer R3.1
- net SDA: no longer R1.1
- net VCC: no longer C5.1, R3.2, R5.2
Other:
- note added: "Non Populated: -"
- note added: "Wireling 0.69 OLED"
- note removed: "0.69" OLED"
- note removed: "Capacitors"
- note removed: "NOTES:"
- note removed: "Non Populated: R1, R2"
- note removed: "SDA and SCL Pull-Up Resistors Optional"
- note removed: "Test R4 with 1.00M, 1.2M, and 820k"
- moved on the sheet: C1, C2, R1, R3
